File: Powersupply/Powersupply.kicad_pcb (KiCad board)
At the start: 2 copper layers, 110 x 31.2 mm, 29 parts, among them J1 Conn_01x02_Pin, J2 Conn_01x02_Pin, Q1 FZT558TA, Q2 FZT458QTA, U1 IRFB9N60APBF, U2 LM431ACM3_NOPB, U3 LM431ACM3_NOPB

Commit message: update
Parts:
- I_SET1: renamed from R3; value 47 -> 39
- V_SET1: renamed from RVset1; value 360k -> 634K
Other:
- board text added: "Danger! High Voltage"
- board text added: "based on changpuak.ch QO-408"
Changed lines of the file:
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@@
 			(drillshape 0)
 			(scaleselection 1)
-			(outputdirectory "")
+			(outputdirectory "Export/")
 		)
 	)
@@
 		(property ki_fp_filters "R_*")
 		(sheetname "/")
-		(sheetfile "200v psu.kicad_sch")
+		(sheetfile "Powersupply.kicad_sch")
 		(attr smd)
 		(fp_line
@@
 		)
 		(sheetname "/")
-		(sheetfile "200v psu.kicad_sch")
+		(sheetfile "Powersupply.kicad_sch")
 		(attr smd)
 		(fp_line
@@
 		(property ki_fp_filters "MountingHole*Pad*")
 		(sheetname "/")
-		(sheetfile "200v psu.kicad_sch")
+		(sheetfile "Powersupply.kicad_sch")
 		(attr exclude_from_pos_files)
 		(fp_circle
@@
 		(property ki_fp_filters "MountingHole*")
 		(sheetname "/")
-		(sheetfile "200v psu.kicad_sch")
+		(sheetfile "Powersupply.kicad_sch")
 		(attr exclude_from_pos_files exclude_from_bom)
 		(pad "" np_thru_hole circle
@@
 		(property ki_fp_filters "C_*")
 		(sheetname "/")
-		(sheetfile "200v psu.kicad_sch")
+		(sheetfile "Powersupply.kicad_sch")
 		(attr through_hole)
 		(fp_line
@@
 		(property ki_fp_filters "MountingHole*")
 		(sheetname "/")
-		(sheetfile "200v psu.kicad_sch")
+		(sheetfile "Powersupply.kicad_sch")
 		(attr exclude_from_pos_files exclude_from_bom)
 		(pad "" np_thru_hole circle
@@
 		(property ki_fp_filters "D*DO?41*")
 		(sheetname "/")
-		(sheetfile "200v psu.kicad_sch")
+		(sheetfile "Powersupply.kicad_sch")
 		(attr smd)
 		(fp_line
@@
 		(property ki_fp_filters "MountingHole*")
 		(sheetname "/")
-		(sheetfile "200v psu.kicad_sch")
+		(sheetfile "Powersupply.kicad_sch")
 		(attr exclude_from_pos_files exclude_from_bom)
 		(pad "" np_thru_hole circle
@@
 		(property ki_fp_filters "R_*")
 		(sheetname "/")
-		(sheetfile "200v psu.kicad_sch")
+		(sheetfile "Powersupply.kicad_sch")
 		(attr smd)
 		(fp_line
@@
 		(descr "Capacitor SMD 0805 (2012 Metric), square (rectangular) end terminal, IPC-7351 nominal with elongated pad for handsoldering. (Body size source: IPC-SM-782 page 76, https://www.pcb-3d.com/wordpress/wp-content/uploads/ipc-sm-782a_amendment_1_and_2.pdf, https://docs.google.com/spreadsheets/d/1BsfQQcO9C6DZCsRaXUlFlo91Tg2WpOkGARC1WS5S8t0/edit?usp=sharing), generated with kicad-footprint-generator")
 		(tags "capacitor handsolder")
-		(property "Reference" "R3"
-			(at 0 -1.68 90)
+		(property "Reference" "I_SET1"
+			(at 2.9275 1.41 180)
 			(layer "F.SilkS")
 			(effects
@@
 			)
 		)
-		(property "Value" "47"
+		(property "Value" "39"
 			(at 0 1.68 90)
 			(layer "F.Fab")
@@
 		(property ki_fp_filters "R_*")
 		(sheetname "/")
-		(sheetfile "200v psu.kicad_sch")
+		(sheetfile "Powersupply.kicad_sch")
 		(attr smd)
 		(fp_line
@@
 		(property ki_fp_filters "MountingHole*")
 		(sheetname "/")
-		(sheetfile "200v psu.kicad_sch")
+		(sheetfile "Powersupply.kicad_sch")
 		(attr exclude_from_pos_files exclude_from_bom)
 		(fp_text user "${REFERENCE}"
@@
 		(property ki_fp_filters "Connector*:*_1x??_*")
 		(sheetname "/")
-		(sheetfile "200v psu.kicad_sch")
+		(sheetfile "Powersupply.kicad_sch")
 		(attr through_hole)
 		(fp_line
@@
 		(property ki_fp_filters "MountingHole*Pad*")
 		(sheetname "/")
-		(sheetfile "200v psu.kicad_sch")
+		(sheetfile "Powersupply.kicad_sch")
 		(attr exclude_from_pos_files)
 		(fp_circle
@@
 		(property ki_fp_filters "D*DO?35*")
 		(sheetname "/")
-		(sheetfile "200v psu.kicad_sch")
+		(sheetfile "Powersupply.kicad_sch")
 		(attr smd)
 		(fp_line
@@
 		(property ki_fp_filters "TO?220*")
 		(sheetname "/")
-		(sheetfile "200v psu.kicad_sch")
+		(sheetfile "Powersupply.kicad_sch")
 		(attr through_hole)
 		(fp_line
@@
 		(property ki_fp_filters "D*DO?41*")
 		(sheetname "/")
-		(sheetfile "200v psu.kicad_sch")
+		(sheetfile "Powersupply.kicad_sch")
 		(attr smd)
 		(fp_line
@@
 		(descr "Capacitor SMD 0805 (2012 Metric), square (rectangular) end terminal, IPC-7351 nominal with elongated pad for handsoldering. (Body size source: IPC-SM-782 page 76, https://www.pcb-3d.com/wordpress/wp-content/uploads/ipc-sm-782a_amendment_1_and_2.pdf, https://docs.google.com/spreadsheets/d/1BsfQQcO9C6DZCsRaXUlFlo91Tg2WpOkGARC1WS5S8t0/edit?usp=sharing), generated with kicad-footprint-generator")
 		(tags "capacitor handsolder")
-		(property "Reference" "RVset1"
-			(at 0 -1.68 0)
+		(property "Reference" "V_SET1"
+			(at -1.82 -2 0)
 			(layer "F.SilkS")
 			(effects
@@
 			)
 		)
-		(property "Value" "360k"
+		(property "Value" "634K"
 			(at 0 1.68 0)
 			(layer "F.Fab")
@@
 		(property ki_fp_filters "R_*")
 		(sheetname "/")
-		(sheetfile "200v psu.kicad_sch")
+		(sheetfile "Powersupply.kicad_sch")
 		(attr smd)
 		(fp_line
@@
 		(property ki_fp_filters "D*DO?35*")
 		(sheetname "/")
-		(sheetfile "200v psu.kicad_sch")
+		(sheetfile "Powersupply.kicad_sch")
 		(attr smd)
 		(fp_line
@@
 		(property ki_fp_filters "R_*")
 		(sheetname "/")
-		(sheetfile "200v psu.kicad_sch")
+		(sheetfile "Powersupply.kicad_sch")
 		(attr smd)
 		(fp_line
@@
 		(property ki_fp_filters "C_*")
 		(sheetname "/")
-		(sheetfile "200v psu.kicad_sch")
+		(sheetfile "Powersupply.kicad_sch")
 		(attr through_hole)
 		(fp_line
@@
 		(property ki_fp_filters "Heatsink_*")
 		(sheetname "/")
-		(sheetfile "200v psu.kicad_sch")
+		(sheetfile "Powersupply.kicad_sch")
 		(attr through_hole)
 		(fp_line
@@
 		(property ki_fp_filters "Connector*:*_1x??_*")
 		(sheetname "/")
-		(sheetfile "200v psu.kicad_sch")
+		(sheetfile "Powersupply.kicad_sch")
 		(attr through_hole)
 		(fp_line
@@
 		(property ki_fp_filters "MountingHole*Pad*")
 		(sheetname "/")
-		(sheetfile "200v psu.kicad_sch")
+		(sheetfile "Powersupply.kicad_sch")
 		(attr exclude_from_pos_files)
 		(fp_circle
@@
 		)
 		(sheetname "/")
-		(sheetfile "200v psu.kicad_sch")
+		(sheetfile "Powersupply.kicad_sch")
 		(attr smd)
 		(fp_line
@@
 		(property ki_fp_filters "Diode*Bridge*OnSemi*SDIP*4L*")
 		(sheetname "/")
-		(sheetfile "200v psu.kicad_sch")
+		(sheetfile "Powersupply.kicad_sch")
 		(attr smd)
 		(fp_line
@@
 		(property ki_fp_filters "R_*")
 		(sheetname "/")
-		(sheetfile "200v psu.kicad_sch")
+		(sheetfile "Powersupply.kicad_sch")
 		(attr smd)
 		(fp_line
@@
 		(property ki_fp_filters "R_*")
 		(sheetname "/")
-		(sheetfile "200v psu.kicad_sch")
+		(sheetfile "Powersupply.kicad_sch")
 		(attr smd)
 		(fp_line
@@
 		)
 		(sheetname "/")
-		(sheetfile "200v psu.kicad_sch")
+		(sheetfile "Powersupply.kicad_sch")
 		(attr smd)
 		(fp_line
@@
 		)
 		(sheetname "/")
-		(sheetfile "200v psu.kicad_sch")
+		(sheetfile "Powersupply.kicad_sch")
 		(attr smd)
 		(fp_line
@@
 		(layer "Edge.Cuts")
 	)
+	(gr_text "based on changpuak.ch QO-408"
+		(at 122.8 112.09 0)
+		(layer "F.SilkS")
+		(effects
+			(font
+				(size 1 1)
+				(thickness 0.15)
+			)
+			(justify left bottom)
+		)
+	)
+	(gr_text "Danger!\nHigh Voltage"
+		(at 168.87 94.42 0)
+		(layer "F.SilkS")
+		(effects
+			(font
+				(size 1 1)
+				(thickness 0.15)
+			)
+			(justify left bottom)
+		)
+	)
 	(segment
