File: Powersupply/Powersupply.kicad_sch (KiCad schematic)
At the start: 29 parts, among them J1 Conn_01x02_Pin, J2 Conn_01x02_Pin, Q1 FZT558TA, Q2 FZT458QTA, U1 IRFB9N60APBF, U2 LM431ACM3_NOPB, U3 LM431ACM3_NOPB

Commit message: update
Parts:
- I_SET1: renamed from R3; value 47 -> 39
- V_SET1: renamed from RVset1; value 360k -> 634K
Other:
- note added: "39ohm = 65mA see https://www.changpuak.ch/electronics/VB408.php to calcualte"
- note added: "634K = 211V see https://www.changpuak.ch/electronics/VB408.php to calcualte"
Changed lines of the file:
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@@
 	(generator_version "9.0")
 	(paper "A4")
+	(text "634K = 211V\n\nsee https://www.changpuak.ch/electronics/VB408.php\nto calcualte\n"
+		(exclude_from_sim no)
+		(at 214.63 97.79 0)
+		(effects
+			(font
+				(size 1.27 1.27)
+			)
+		)
+	)
+	(text "39ohm = 65mA\n\nsee https://www.changpuak.ch/electronics/VB408.php\nto calcualte\n"
+		(exclude_from_sim no)
+		(at 173.99 25.4 0)
+		(effects
+			(font
+				(size 1.27 1.27)
+			)
+		)
+	)
 	(junction
 		(at 167.64 102.87)
@@
 		(dnp no)
 		(fields_autoplaced yes)
-		(property "Reference" "R3"
+		(property "Reference" "I_SET1"
 			(at 166.37 33.02 90)
 			(effects
@@
 			)
 		)
-		(property "Value" "47"
+		(property "Value" "39"
 			(at 166.37 35.56 90)
 			(effects
@@
 			(project "Untitled"
 				(path "/993c4fa3-eb3b-4c54-a665-861e22316333"
-					(reference "R3")
+					(reference "I_SET1")
 					(unit 1)
 				)
@@
 		(dnp no)
 		(fields_autoplaced yes)
-		(property "Reference" "RVset1"
+		(property "Reference" "V_SET1"
 			(at 181.61 96.5199 0)
 			(effects
@@
 			)
 		)
-		(property "Value" "360k"
+		(property "Value" "634K"
 			(at 181.61 99.0599 0)
 			(effects
@@
 			(project "Untitled"
 				(path "/993c4fa3-eb3b-4c54-a665-861e22316333"
-					(reference "RVset1")
+					(reference "V_SET1")
 					(unit 1)
 				)
