File: Amplifier Compound/Amplifier Compound.kicad_sch (KiCad schematic)
At the start: 46 parts, among them J1 Screw_Terminal_01x02, J3 Screw_Terminal_01x02, U1 PA88

Commit message: compound
Parts:
- added C10, C6, C7: 15pF, Capacitor_SMD:C_1206_3216Metric_Pad1.33x1.80mm_HandSolder, symbol Device:C_Small
- added C8, C9: 0.1u, Capacitor_SMD:C_1206_3216Metric_Pad1.33x1.80mm_HandSolder, symbol Device:C_Small
- added U2: LT1012, Package_SO:SOIC-8_3.9x4.9mm_P1.27mm, symbol Amplifier_Operational:LT1012
- C2, C5: footprint Capacitor_SMD:C_1206_3216Metric_Pad1.33x1.80mm_HandSolder -> Capacitor_SMD:CP_Elec_6.3x7.7
- D5, D6: value D_Zener 6.2V -> D_Zener 15V
- R10: value 220k -> 100k; Part Description RES SMD 16.9K OHM 1% 1/4W 1206 -> (none)
- R13: value 220k -> 11k; Part Description RES SMD 16.9K OHM 1% 1/4W 1206 -> (none)
- R3: value 330k -> 100k; Part Description RES SMD 16.9K OHM 1% 1/4W 1206 -> (none)
Connections:
- net +VLV: now also RV2.2, C9.2, U2.7 (V+); no longer R10.2
- net -VLV: now also C8.2, U2.4 (V-); no longer R13.1
- net CTRL: now also U2.6; no longer J3.1 (Pin_1), R17.1
- net GND: now also R13.2, C7.1, C8.1, C9.1
- net HVOUT: now also R10.1, C10.2, C6.2
- net at D1.2 (A), D2.1 (K), U1.5 (-IN): now also R13.1, R3.2, C10.1; no longer R16.2, RV1.1
- net at RV2.1: now also U2.8 (C/B); no longer R10.1
- net at R2.2, R7.1: no longer R3.1
- net at RV2.3: now also U2.1 (BAL); no longer R13.2
- net at R19.1, RV1.2: now also RV1.1; no longer RV1.3
- new net: C7.2, U2.5 (COMP)
- new net: C6.1, R16.2, RV1.3, U2.2 (-)
- new net: R10.2, R3.1
- new net: J3.1 (Pin_1), R17.1, U2.3 (+)
Other:
- moved on the sheet: C3, C5, D3, D5, J3, R15, R16, R17, R18, R19, R2, R20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

Commit message: update
Other:
- moved on the sheet: C2, C5, C8, C9, D5, D6, J3, R11, R12, R14, R15, R17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
