File: Amplifier Compound/Amplifier Compound.kicad_sch (KiCad schematic)
At the start: 52 parts, among them J1 Screw_Terminal_01x02, J3 Screw_Terminal_01x02, U1 PA88, U2 LT1012

Commit message: update composite
Parts:
- removed D1, D2: DSS120U, Diode_SMD:D_SOD-123F, symbol Device:D_Small
- added D16: SMA6J12CA, Diode_SMD:D_SMA_Handsoldering, symbol Device:D_TVS
- added Q1, Q2: MMBF5457, Package_TO_SOT_SMD:SOT-23-3, symbol Simulation_SPICE:NJFET
- added R21: 10k, Resistor_SMD:R_1206_3216Metric_Pad1.30x1.75mm_HandSolder, symbol Device:R_Small_US
- added R22: 220k, Resistor_THT:R_Axial_DIN0411_L9.9mm_D3.6mm_P5.08mm_Vertical, symbol Device:R_Small_US
- added TP5: GND, TestPoint:TestPoint_THTPad_2.5x2.5mm_Drill1.2mm, symbol jmlib:tp_small
- C10, C6: value 15pF -> 6.6pF; Part Description CAP CER 15PF 50V C0G/NP0 1206 -> CAP CER 15PF 450V C0G/NP0 1206; Voltage 50V -> 450V
- C2: value 200pf -> 100uf; Package 1206 -> (none); Part Description CAP CER 0.1UF 450V X7T 1206 -> (none); Voltage 450V -> 25v
- C5: value 200pf -> 100uf; Package 1206 -> (none); Part Description CAP CER 0.1UF 450V X7T 1206 -> (none); Voltage 450V -> 24v
- C7: value 15pF -> 160pf
- D5, D6: value D_Zener 15V -> D_Zener 18V; footprint Diode_SMD:D_MiniMELF -> Diode_THT:D_A-405_P10.16mm_Horizontal
- H1, H2, H3, H4: footprint MountingHole:MountingHole_3.2mm_M3_DIN965_Pad -> MountingHole:MountingHole_3.2mm_M3_DIN965_Pad_TopBottom
- J1, J3: footprint Connector_Phoenix_MC:PhoenixContact_MCV_1,5_2-G-3.5_1x02_P3.50mm_Vertical -> Connector_Molex:Molex_KK-396_A-41791-0002_1x02_P3.96mm_Vertical
- R11, R12, R14: value 68k -> 220k; footprint Resistor_SMD:R_1206_3216Metric_Pad1.30x1.75mm_HandSolder -> Resistor_THT:R_Axial_DIN0411_L9.9mm_D3.6mm_P5.08mm_Vertical
- R15: value 68k -> 10k; Part Description RES SMD 16.9K OHM 1% 1/4W 1206 -> RES SMD 100 OHM 1% 1/4W 1206
- R17: value NC -> 10M
- R8: value 68k -> 100R; Part Description RES SMD 16.9K OHM 1% 1/4W 1206 -> (none)
- R9: value 68K -> 100R; Part Description RES SMD 16.9K OHM 1% 1/4W 1206 -> (none)
- U2: footprint Package_SO:SOIC-8_3.9x4.9mm_P1.27mm -> Package_DIP:DIP-8_W7.62mm_LongPads
Connections:
- net +VHV: now also R12.2; no longer R15.2
- net +VLV: now also C5.1, R14.1; no longer C5.2, R9.1
- net -VHV: now also R22.2; no longer R11.2
- net -VLV: now also R11.1; no longer R12.1
- net CTRL: now also R21.1; no longer U1.4 (+IN)
- net GND: now also C5.2, H2.1, H4.1, R17.1, D16.1 (A1), TP5.1; no longer C5.1, R17.2
- net HVOUT: now also R8.1, R9.1; no longer C10.2, C6.2
- net at C10.1, R13.1, R3.2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: now also Q1.1 (D), Q1.2 (S), Q2.3 (G)
- net at R15.1: now also U2.3 (+); no longer R8.2
- net at R14.2: now also R12.1; no longer R11.1
- net at R9.2: now also C10.2; no longer R8.1
- new net: R11.2, R22.1
- new net: Q1.3 (G), Q2.1 (D), Q2.2 (S), R21.2, U1.4 (+IN)
- new net: D16.2 (A2), J3.1 (Pin_1), R15.2, R17.2
- new net: C6.2, R8.2
Other:
- moved on the sheet: C1, C10, C3, C5, C6, C7, D3, J3, R1, R10, R13, R16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

Commit message: final components update
Parts:
- added R23: 100, Resistor_SMD:R_1206_3216Metric_Pad1.30x1.75mm_HandSolder, symbol Device:R_Small_US
Connections:
- net HVOUT: now also R23.1; no longer R10.1, R5.1, R6.1, R8.1, R9.1, U1.1 (OUT)
- new net: R10.1, R23.2, R5.1, R6.1, R8.1, R9.1, U1.1 (OUT)
Changed lines of the file:
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@@
 	(wire
 		(pts
-			(xy 177.8 85.09) (xy 200.66 85.09)
+			(xy 177.8 85.09) (xy 182.88 85.09)
 		)
 		(stroke
@@
 	(wire
 		(pts
+			(xy 187.96 85.09) (xy 200.66 85.09)
+		)
+		(stroke
+			(width 0)
+			(type default)
+		)
+	)
+	(wire
+		(pts
 			(xy 111.76 177.8) (xy 111.76 179.07)
 		)
@@
 					(unit 1)
 				)
+			)
+		)
+	)
+	(symbol
+		(lib_id "Device:R_Small_US")
+		(at 185.42 85.09 270)
+		(unit 1)
+		(exclude_from_sim no)
+		(in_bom yes)
+		(on_board yes)
+		(dnp no)
+		(property "Reference" "R23"
+			(at 184.15 82.55 90)
+			(effects
+				(font
+					(size 1.27 1.27)
+				)
+				(justify left)
+			)
+		)
+		(property "Value" "100"
+			(at 184.15 87.63 90)
+			(effects
+				(font
+					(size 1.27 1.27)
+				)
+				(justify left)
+			)
+		)
+		(property "Footprint" "Resistor_SMD:R_1206_3216Metric_Pad1.30x1.75mm_HandSolder"
+			(at 185.42 85.09 0)
+			(effects
+				(font
+					(size 1.27 1.27)
+				)
+				(hide yes)
+			)
+		)
+		(property "Datasheet" "~"
+			(at 185.42 85.09 0)
+			(effects
+				(font
+					(size 1.27 1.27)
+				)
+				(hide yes)
+			)
+		)
+		(property "Description" "11ohm for max 64mA R=0,7/I"
+			(at 197.485 90.17 90)
+			(effects
+				(font
+					(size 1.27 1.27)
+				)
+				(hide yes)
+			)
+		)
+		(property "Package" "1206"
+			(at 185.42 85.09 0)
+			(effects
+				(font
+					(size 1.27 1.27)
+				)
+				(hide yes)
+			)
+		)
+		(property "Part Description" "RES 150 OHM 1% 1/2W 1206"
+			(at 185.42 85.09 0)
+			(effects
+				(font
+					(size 1.27 1.27)
+				)
+				(hide yes)
+			)
+		)
+		(pin "1"
+		)
+		(pin "2"
+		)
+		(instances
+			(project "Amplifier Compound"
+				(path "/e63e39d7-6ac0-4ffd-8aa3-1841a4541b55"
+					(reference "R23")
+					(unit 1)
+				)

Commit message: extra feedback
Parts:
- added C11: 100pf, Capacitor_SMD:C_1206_3216Metric_Pad1.33x1.80mm_HandSolder, symbol Device:C_Small
- added R24: 100R, Resistor_SMD:R_1206_3216Metric_Pad1.30x1.75mm_HandSolder, symbol Device:R_Small_US
- C7: value 160pf -> 68pf
Connections:
- net CTRL: now also C11.1
- net at C6.1, R16.2, RV1.3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: now also R24.1
- new net: C11.2, R24.2
