File: Amplifier Compound/Amplifier Compound.kicad_pcb (KiCad board)
At the start: 2 copper layers, 77.7 x 60 mm, 52 parts, among them J1 Screw_Terminal_01x02, J3 Screw_Terminal_01x02, U1 PA88, U2 LT1012

Commit message: update
Parts:
- moved R14 0.64 mm to (140.6, 106.4)
Routing:
- net +VLV: track 98.7 -> 93.8 mm
- net -VLV: track 75.8 -> 72.8 mm
Changed lines of the file:
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@@
 	(footprint "Resistor_SMD:R_1206_3216Metric_Pad1.30x1.75mm_HandSolder"
 		(layer "F.Cu")
-		(at 140.07 106.73 180)
+		(at 140.63 106.43 180)
 		(descr "Resistor SMD 1206 (3216 Metric), square (rectangular) end terminal, IPC-7351 nominal with elongated pad for handsoldering. (Body size source: IPC-SM-782 page 72, https://www.pcb-3d.com/wordpress/wp-content/uploads/ipc-sm-782a_amendment_1_and_2.pdf), generated with kicad-footprint-generator")
 		(tags "resistor handsolder")
@@
 	)
 	(segment
-		(start 141.98 95.479999)
-		(end 138.490001 91.99)
+		(start 168.339 81.989)
+		(end 171.76 85.41)
 		(width 1)
 		(layer "F.Cu")
@@
 	(segment
 		(start 141.98 95.479999)
-		(end 147.220001 95.479999)
+		(end 138.490001 91.99)
 		(width 1)
 		(layer "F.Cu")
@@
 	)
 	(segment
-		(start 142.26 99.71)
-		(end 142.3 99.75)
-		(width 0.5)
+		(start 158.711 81.989)
+		(end 168.339 81.989)
+		(width 1)
 		(layer "F.Cu")
 		(net 9)
 	)
 	(segment
-		(start 160.711 81.989)
-		(end 168.339 81.989)
+		(start 141.98 95.479999)
+		(end 145.220001 95.479999)
 		(width 1)
 		(layer "F.Cu")
@@
 	)
 	(segment
-		(start 147.220001 95.479999)
-		(end 160.711 81.989)
+		(start 142.26 99.71)
+		(end 142.3 99.75)
+		(width 0.5)
+		(layer "F.Cu")
+		(net 9)
+	)
+	(segment
+		(start 145.220001 95.479999)
+		(end 158.711 81.989)
 		(width 1)
 		(layer "F.Cu")
@@
 	)
 	(segment
-		(start 168.339 81.989)
-		(end 171.76 85.41)
-		(width 1)
-		(layer "F.Cu")
-		(net 9)
-	)
-	(segment
 		(start 171.548319 90.9753)
 		(end 173.680552 88.843067)
@@
 	)
 	(segment
-		(start 150.36 67.29)
-		(end 168.88 67.29)
-		(width 1)
-		(layer "F.Cu")
-		(net 10)
-	)
-	(segment
 		(start 132.11 101.03)
 		(end 135.05 103.97)
@@
 	)
 	(segment
-		(start 149.380001 68.269999)
-		(end 150.36 67.29)
-		(width 1)
-		(layer "F.Cu")
-		(net 10)
-	)
-	(segment
 		(start 133.63 76.74)
 		(end 132.11 78.26)
@@
 	)
 	(segment
-		(start 141.92 75.740001)
-		(end 149.380001 68.28)
+		(start 147.559999 75.740001)
+		(end 156.01 67.29)
 		(width 1)
 		(layer "F.Cu")
@@
 	)
 	(segment
-		(start 132.11 78.26)
-		(end 132.11 101.03)
-		(width 0.5)
+		(start 141.92 75.740001)
+		(end 147.559999 75.740001)
+		(width 1)
 		(layer "F.Cu")
 		(net 10)
 	)
 	(segment
-		(start 168.88 67.29)
-		(end 171.76 70.17)
+		(start 156.01 67.29)
+		(end 168.88 67.29)
 		(width 1)
 		(layer "F.Cu")
@@
 	)
 	(segment
+		(start 132.11 78.26)
+		(end 132.11 101.03)
+		(width 0.5)
+		(layer "F.Cu")
+		(net 10)
+	)
+	(segment
 		(start 135.43 76.74)
 		(end 140.920001 76.74)
@@
 	)
 	(segment
-		(start 149.380001 68.28)
-		(end 149.380001 68.269999)
+		(start 168.88 67.29)
+		(end 171.76 70.17)
 		(width 1)
 		(layer "F.Cu")
@@
 	)
 	(segment
-		(start 199.06 110.82)
-		(end 199.06 110.351364)
+		(start 184.31 110.83)
+		(end 199.05 110.83)
+		(width 0.5)
+		(layer "F.Cu")
+		(net 14)
+	)
+	(segment
+		(start 195.7435 88.469)
+		(end 194.4375 89.775)
 		(width 0.5)
 		(layer "F.Cu")
@@
 	)
 	(segment
-		(start 160.16 116.92)
-		(end 159.24 116)
+		(start 199.05 110.83)
+		(end 201.091 108.789)
 		(width 0.5)
 		(layer "F.Cu")
@@
 	)
 	(segment
-		(start 182.62 116.92)
-		(end 160.16 116.92)
+		(start 198.337292 88.469)
+		(end 195.7435 88.469)
 		(width 0.5)
 		(layer "F.Cu")
@@
 	)
 	(segment
-		(start 184.31 115.23)
-		(end 182.62 116.92)
+		(start 159.24 112.4)
+		(end 159.24 109.69)
 		(width 0.5)
 		(layer "F.Cu")
@@
 	)
 	(segment
-		(start 156.04 99.75)
-		(end 156.04 96.0025)
+		(start 184.31 112.82)
+		(end 181.85 115.28)
 		(width 0.5)
 		(layer "F.Cu")
@@
 	)
 	(segment
-		(start 184.31 110.83)
-		(end 184.31 115.23)
+		(start 162.12 115.28)
+		(end 159.24 112.4)
 		(width 0.5)
 		(layer "F.Cu")
@@
 	)
 	(segment
-		(start 201.091 108.320364)
-		(end 201.091 96.639636)
+		(start 156.04 99.75)
+		(end 156.04 96.0025)
 		(width 0.5)
 		(layer "F.Cu")
@@
 	)
 	(segment
-		(start 201.091 96.639636)
-		(end 199.06 94.608636)
+		(start 199.06 94.608636)
+		(end 199.06 89.191708)
 		(width 0.5)
 		(layer "F.Cu")
@@
 	)
 	(segment
-		(start 199.05 110.83)
-		(end 199.06 110.82)
+		(start 201.091 108.789)
+		(end 201.091 96.639636)
 		(width 0.5)
 		(layer "F.Cu")
@@
 	)
 	(segment
-		(start 198.337292 88.469)
-		(end 199.06 89.191708)
+		(start 181.85 115.28)
+		(end 162.12 115.28)
 		(width 0.5)
 		(layer "F.Cu")
@@
 	)
 	(segment
-		(start 194.4375 89.775)
-		(end 195.7435 88.469)
-		(width 0.5)
-		(layer "F.Cu")
-		(net 14)
-	)
-	(segment
 		(start 184.31 110.83)
-		(end 199.05 110.83)
+		(end 184.31 112.82)
 		(width 0.5)
 		(layer "F.Cu")
@@
 	)
 	(segment
-		(start 159.24 116)
-		(end 159.24 109.69)
-		(width 0.5)
-		(layer "F.Cu")
-		(net 14)
-	)
-	(segment
-		(start 195.7435 88.469)
+		(start 199.06 89.191708)
 		(end 198.337292 88.469)
 		(width 0.5)
@@
 	)
 	(segment
-		(start 199.06 89.191708)
+		(start 201.091 96.639636)
 		(end 199.06 94.608636)
 		(width 0.5)
@@
 	)
 	(segment
-		(start 199.06 110.351364)
-		(end 201.091 108.320364)
-		(width 0.5)
-		(layer "F.Cu")
-		(net 14)
-	)
-	(segment
-		(start 192.4 118.28)
-		(end 159.26 118.28)
+		(start 195.71 112.42)
+		(end 191.64 116.49)
 		(width 0.5)
 		(layer "F.Cu")
@@
 	)
 	(segment
-		(start 195.71 114.97)
-		(end 192.4 118.28)
+		(start 157.5 116.49)
+		(end 153.84 112.83)
 		(width 0.5)
 		(layer "F.Cu")
@@
 	)
 	(segment
-		(start 146.65 112.7075)
+		(start 153.84 112.83)
 		(end 146.7725 112.83)
 		(width 0.5)
@@
 	)
 	(segment
-		(start 146.7725 112.83)
-		(end 153.81 112.83)
-		(width 0.5)
-		(layer "F.Cu")
-		(net 15)
-	)
-	(segment
-		(start 147.05 109.06)
-		(end 146.65 108.66)
+		(start 195.71 111.88)
+		(end 195.71 112.42)
 		(width 0.5)
 		(layer "F.Cu")
@@
 	)
 	(segment
-		(start 146.65 108.66)
-		(end 146.65 112.7075)
+		(start 191.64 116.49)
+		(end 157.5 116.49)
 		(width 0.5)
 		(layer "F.Cu")
@@
 	)
 	(segment
-		(start 159.26 118.28)
-		(end 156.46 115.48)
+		(start 146.65 112.7075)
+		(end 146.65 108.66)
 		(width 0.5)
 		(layer "F.Cu")
@@
 	)
 	(segment
-		(start 195.71 111.88)
-		(end 195.71 114.97)
+		(start 146.65 108.66)
+		(end 147.05 109.06)
 		(width 0.5)
 		(layer "F.Cu")
@@
 	)
 	(segment
-		(start 153.81 112.83)
-		(end 156.46 115.48)
+		(start 146.7725 112.83)
+		(end 146.65 112.7075)
 		(width 0.5)
 		(layer "F.Cu")
@@
 	)
 	(segment
-		(start 138.15 106.36)
-		(end 138.52 106.73)
+		(start 138.15 105.5)
+		(end 139.08 106.43)
 		(width 0.5)
 		(layer "F.Cu")
@@
 	(segment
 		(start 138.15 103.97)
-		(end 138.15 106.36)
+		(end 138.15 105.5)
 		(width 0.5)
 		(layer "F.Cu")
@@
 	)
 	(segment
-		(start 141.62 106.73)
-		(end 141.68 106.73)
+		(start 142.18 107.23)
+		(end 143.71 108.76)
 		(width 0.5)
 		(layer "F.Cu")
@@
 	)
 	(segment
-		(start 141.68 106.73)
-		(end 143.71 108.76)
+		(start 142.18 106.43)
+		(end 142.18 107.23)
 		(width 0.5)
 		(layer "F.Cu")

Commit message: update composite
Parts:
- removed D1, D2: DSS120U, Diode_SMD:D_SOD-123F
- added D16: SMA6J12CA, Diode_SMD:D_SMA_Handsoldering, F.Cu at (199.7, 82.7)
- added Q1: MMBF5457, Package_TO_SOT_SMD:SOT-23-3, B.Cu at (180.1, 87.2)
- added Q2: MMBF5457, Package_TO_SOT_SMD:SOT-23-3, B.Cu at (177.6, 84.6)
- added R21: 10k, Resistor_SMD:R_1206_3216Metric_Pad1.30x1.75mm_HandSolder, F.Cu at (186.8, 89.0)
- added R22: 220k, Resistor_THT:R_Axial_DIN0411_L9.9mm_D3.6mm_P5.08mm_Vertical, F.Cu at (122.6, 87.0)
- added TP5: GND, TestPoint:TestPoint_THTPad_2.5x2.5mm_Drill1.2mm, F.Cu at (206.3, 111.5)
- C10, C6: value 15pF -> 6.6pF
- C2, C5: value 200pf -> 100uf
- C7, C8, C9: moved to B.Cu
- D5, D6: value D_Zener 15V -> D_Zener 18V; footprint Diode_SMD:D_MiniMELF -> Diode_THT:D_A-405_P10.16mm_Horizontal
- H1, H2, H3, H4: footprint MountingHole:MountingHole_3.2mm_M3_DIN965_Pad -> MountingHole:MountingHole_3.2mm_M3_ISO7380_Pad
- J1, J3: footprint Connector_Phoenix_MC:PhoenixContact_MCV_1,5_2-G-3.5_1x02_P3.50mm_Vertical -> Connector_Molex:Molex_KK-396_A-41791-0002_1x02_P3.96mm_Vertical
- R11, R12, R14: value 68k -> 220k; footprint Resistor_SMD:R_1206_3216Metric_Pad1.30x1.75mm_HandSolder -> Resistor_THT:R_Axial_DIN0411_L9.9mm_D3.6mm_P5.08mm_Vertical
- R15: value 68k -> 10k
- R17: value NC -> 10M; moved to B.Cu
- R8: value 68k -> 100R
- R9: value 68K -> 100R; moved to B.Cu
- U2: footprint Package_SO:SOIC-8_3.9x4.9mm_P1.27mm -> Package_DIP:DIP-8_W7.62mm_LongPads
- moved R15 64.2 mm to (206.1, 84.1), turned to 90 degrees
- moved C2 36.5 mm to (190.3, 116.9)
- moved TP4 33.4 mm to (122.0, 118.3), turned to 180 degrees
- moved C5 28.2 mm to (180.0, 117.0)
- moved TP1 27.8 mm to (126.8, 118.4), turned to 180 degrees
- moved R12 23.8 mm to (122.4, 102.3), turned to 0 degrees
- moved R8 20.8 mm to (169.9, 97.2), turned to 0 degrees
- moved TP3 20.2 mm to (122.4, 65.5), turned to -90 degrees
- moved D5 20.2 mm to (138.3, 108.4), turned to 0 degrees
- moved R9 19.8 mm to (161.8, 81.3), turned to 45 degrees
- moved R14 16.6 mm to (126.9, 97.1)
- moved R11 15.8 mm to (127.0, 91.5)
- moved TP2 14.1 mm to (127.0, 65.5), turned to -90 degrees
- moved R13 12.0 mm to (177.7, 78.5)
- moved D6 10.9 mm to (145.0, 102.0), turned to 180 degrees
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Connections:
- C10 pad 2: /HVOUT -> Net-(C10-Pad2)
- C5 pad 1: GND -> +VLV
- C5 pad 2: +VLV -> GND
- C6 pad 2: /HVOUT -> Net-(C6-Pad2)
- H2 pad 1: unconnected-(H2-Pad1) -> GND
- H4 pad 1: unconnected-(H4-Pad1) -> GND
- J3 pad 1: Net-(J3-Pin_1) -> Net-(D16-A2)
- R11 pad 1: Net-(R11-Pad1) -> -VLV
- R11 pad 2: -VHV -> Net-(R11-Pad2)
- R12 pad 1: -VLV -> Net-(R12-Pad1)
- R12 pad 2: Net-(R12-Pad2) -> +VHV
- R14 pad 1: Net-(R12-Pad2) -> +VLV
- R14 pad 2: Net-(R11-Pad1) -> Net-(R12-Pad1)
- R15 pad 1: Net-(R15-Pad1) -> Net-(U2-+)
- R15 pad 2: +VHV -> Net-(D16-A2)
- R17 pad 1: Net-(J3-Pin_1) -> GND
- R17 pad 2: GND -> Net-(D16-A2)
- R8 pad 1: Net-(R8-Pad1) -> /HVOUT
- R8 pad 2: Net-(R15-Pad1) -> Net-(C6-Pad2)
- R9 pad 1: +VLV -> /HVOUT
- R9 pad 2: Net-(R8-Pad1) -> Net-(C10-Pad2)
- U1 pad 4: /CTRL -> Net-(Q1-G)
- U2 pad 3: Net-(J3-Pin_1) -> Net-(U2-+)
Routing:
- net Net-(J3-Pin_1): track 29.1 -> 0.00 mm, vias 2 -> 0
- net -VLV: track 72.8 -> 101.9 mm, vias 2 -> 3
- net +VHV: track 57.2 -> 83.5 mm
- net GND: track 27.1 -> 2.73 mm, vias 7 -> 90
- net +VLV: track 93.8 -> 113.2 mm
- net Net-(U2-BAL): track 28.6 -> 13.7 mm
- net /HVOUT: track 54.0 -> 39.2 mm
- net Net-(Q1-G): track 0.00 -> 14.3 mm, vias 0 -> 1
- net Net-(U2-+): track 0.00 -> 13.7 mm, vias 0 -> 1
- net /CTRL: track 27.9 -> 14.8 mm, vias 1 -> 0
- net Net-(D16-A2): track 0.00 -> 12.4 mm
- net Net-(C6-Pad2): track 0.00 -> 9.41 mm
- net Net-(U2--): track 20.2 -> 27.3 mm
- net Net-(R11-Pad2): track 0.00 -> 4.84 mm
- net Net-(R12-Pad1): track 0.00 -> 4.80 mm
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- added copper zone on F.Cu, net GND
Other:
- board size 77.7 x 60 mm -> 90 x 60 mm
- board text added: "HV +"
- board text added: "HV -"
- board text added: "High Voltage Danger!"
- board text added: "LV +"
- board text added: "LV -"
- board text removed: "+VHV"
- board text removed: "-VHV"

Commit message: final components update
Parts:
- added R23: 100, Resistor_SMD:R_1206_3216Metric_Pad1.30x1.75mm_HandSolder, F.Cu at (160.3, 105.1)
- C7: value 15pF -> 160pf
Connections:
- R10 pad 1: /HVOUT -> Net-(U1-OUT)
- R5 pad 1: /HVOUT -> Net-(U1-OUT)
- R6 pad 1: /HVOUT -> Net-(U1-OUT)
- R8 pad 1: /HVOUT -> Net-(U1-OUT)
- R9 pad 1: /HVOUT -> Net-(U1-OUT)
- U1 pad 1: /HVOUT -> Net-(U1-OUT)
Routing:
- net Net-(U1-OUT): track 0.00 -> 34.5 mm
- net /HVOUT: track 39.2 -> 4.88 mm

Commit message: clearance
Parts:
- moved R13 2.23 mm to (178.3, 76.4)
- moved R10 0.44 mm to (160.6, 79.2)
Routing:
- net Net-(Q1-D): track 20.6 -> 22.5 mm

Commit message: extra feedback
Parts:
- added C11: 100pf, Capacitor_SMD:C_1206_3216Metric_Pad1.33x1.80mm_HandSolder, B.Cu at (192.2, 88.5)
- added R24: 100R, Resistor_SMD:R_1206_3216Metric_Pad1.30x1.75mm_HandSolder, B.Cu at (190.1, 94.7)
- C7: value 160pf -> 68pf
Routing:
- net Net-(C11-Pad2): track 0.00 -> 3.93 mm
- net Net-(U2--): vias 0 -> 1
- net GND: vias 90 -> 94
- net /CTRL: vias 0 -> 1
